Commit message: Add main robot URDF xacro file

File: mars_robots/urdf/mars_robot.urdf.xacro (robot description, xacro)
@@ -1,197 +1,162 @@
 <?xml version="1.0"?>
 <robot xmlns:xacro="http://www.ros.org/wiki/xacro" name="mars_robot">
-  <!-- Include the differential drive plugin -->
-  <xacro:include filename="$(find mars_robots)/urdf/mars_robot.gazebo.xacro" />
+  <!-- Include Gazebo configurations -->
+  <xacro:include filename="$(find mars_robots)/urdf/mars_robot.gazebo.xacro"/>
   <!-- Robot Properties -->
-  <xacro:property name="chassis_length" value="0.5" />
-  <xacro:property name="chassis_width" value="0.3" />
-  <xacro:property name="chassis_height" value="0.15" />
-  <xacro:property name="chassis_mass" value="5.0" />
-  <xacro:property name="wheel_radius" value="0.1" />
-  <xacro:property name="wheel_width" value="0.05" />
-  <xacro:property name="wheel_mass" value="0.5" />
-  <xacro:property name="wheel_offset_x" value="0.15" />
-  <xacro:property name="wheel_offset_y" value="0.175" />
-  <xacro:property name="wheel_offset_z" value="0.0" />
-  <xacro:property name="caster_radius" value="0.05" />
-  <xacro:property name="caster_mass" value="0.5" />
-  <!-- Base Footprint Link -->
-  <link name="$(arg robot_namespace)/base_footprint"/>
+  <xacro:property name="base_width" value="0.3"/>
+  <xacro:property name="base_length" value="0.3"/>
+  <xacro:property name="base_height" value="0.15"/>
+  <xacro:property name="wheel_radius" value="0.05"/>
+  <xacro:property name="wheel_width" value="0.04"/>
+  <xacro:property name="wheel_separation" value="0.25"/>
+  <xacro:property name="wheel_offset_z" value="-0.05"/>
+  <xacro:property name="caster_radius" value="0.025"/>
   <!-- Base Link -->
-  <link name="$(arg robot_namespace)/base_link">
+  <link name="base_link">
+    <visual>
+      <geometry>
+        <box size="${base_length} ${base_width} ${base_height}"/>
+      </geometry>
+      <material name="red">
+        <color rgba="1 0 0 1"/>
+      </material>
+    </visual>
     <collision>
-      <origin xyz="0 0 ${chassis_height/2}" rpy="0 0 0"/>
       <geometry>
-        <box size="${chassis_length} ${chassis_width} ${chassis_height}"/>
+        <box size="${base_length} ${base_width} ${base_height}"/>
       </geometry>
     </collision>
+    <inertial>
+      <mass value="5.0"/>
+      <inertia ixx="0.1" ixy="0" ixz="0" iyy="0.1" iyz="0" izz="0.1"/>
+    </inertial>
+  </link>
+  <!-- Left Wheel -->
+  <link name="left_wheel">
     <visual>
-      <origin xyz="0 0 ${chassis_height/2}" rpy="0 0 0"/>
       <geometry>
-        <box size="${chassis_length} ${chassis_width} ${chassis_height}"/>
+        <cylinder radius="${wheel_radius}" length="${wheel_width}"/>
       </geometry>
-      <material name="red">
-        <color rgba="0.8 0.2 0.2 1.0"/>
+      <material name="black">
+        <color rgba="0 0 0 1"/>
       </material>
     </visual>
-    <inertial>
-      <origin xyz="0 0 ${chassis_height/2}" rpy="0 0 0"/>
-      <mass value="${chassis_mass}"/>
-      <inertia
-        ixx="${chassis_mass/12.0 * (chassis_width*chassis_width + chassis_height*chassis_height)}"
-        ixy="0.0"
-        ixz="0.0"
-        iyy="${chassis_mass/12.0 * (chassis_length*chassis_length + chassis_height*chassis_height)}"
-        iyz="0.0"
-        izz="${chassis_mass/12.0 * (chassis_length*chassis_length + chassis_width*chassis_width)}"/>
-    </inertial>
-  </link>
-  <!-- Base Footprint to Base Link Joint -->
-  <joint name="$(arg robot_namespace)/base_footprint_joint" type="fixed">
-    <parent link="$(arg robot_namespace)/base_footprint"/>
-    <child link="$(arg robot_namespace)/base_link"/>
-    <origin xyz="0 0 ${wheel_radius}" rpy="0 0 0"/>
-  </joint>
-  <!-- Left Wheel Link -->
-  <link name="$(arg robot_namespace)/left_wheel">
     <collision>
-      <origin xyz="0 0 0" rpy="${pi/2} 0 0"/>
       <geometry>
         <cylinder radius="${wheel_radius}" length="${wheel_width}"/>
       </geometry>
     </collision>
+    <inertial>
+      <mass value="0.5"/>
+      <inertia ixx="0.01" ixy="0" ixz="0" iyy="0.01" iyz="0" izz="0.01"/>
+    </inertial>
+  </link>
+  <!-- Right Wheel -->
+  <link name="right_wheel">
     <visual>
-      <origin xyz="0 0 0" rpy="${pi/2} 0 0"/>
       <geometry>
         <cylinder radius="${wheel_radius}" length="${wheel_width}"/>
       </geometry>
       <material name="black">
-        <color rgba="0.1 0.1 0.1 1.0"/>
+        <color rgba="0 0 0 1"/>
       </material>
     </visual>
-    <inertial>
-      <origin xyz="0 0 0" rpy="${pi/2} 0 0"/>
-      <mass value="${wheel_mass}"/>
-      <inertia
-        ixx="${wheel_mass/12.0 * (3*wheel_radius*wheel_radius + wheel_width*wheel_width)}"
-        ixy="0.0"
-        ixz="0.0"
-        iyy="${wheel_mass/12.0 * (3*wheel_radius*wheel_radius + wheel_width*wheel_width)}"
-        iyz="0.0"
-        izz="${wheel_mass/2.0 * wheel_radius*wheel_radius}"/>
-    </inertial>
-  </link>
-  <!-- Left Wheel Joint -->
-  <joint name="$(arg robot_namespace)/left_wheel_joint" type="continuous">
-    <parent link="$(arg robot_namespace)/base_link"/>
-    <child link="$(arg robot_namespace)/left_wheel"/>
-    <origin xyz="${wheel_offset_x} ${wheel_offset_y} ${wheel_offset_z}" rpy="0 0 0"/>
-    <axis xyz="0 1 0"/>
-  </joint>
-  <!-- Right Wheel Link -->
-  <link name="$(arg robot_namespace)/right_wheel">
     <collision>
-      <origin xyz="0 0 0" rpy="${pi/2} 0 0"/>
       <geometry>
         <cylinder radius="${wheel_radius}" length="${wheel_width}"/>
       </geometry>
     </collision>
+    <inertial>
+      <mass value="0.5"/>
+      <inertia ixx="0.01" ixy="0" ixz="0" iyy="0.01" iyz="0" izz="0.01"/>
+    </inertial>
+  </link>
+  <!-- Front Caster -->
+  <link name="front_caster">
     <visual>
-      <origin xyz="0 0 0" rpy="${pi/2} 0 0"/>
       <geometry>
-        <cylinder radius="${wheel_radius}" length="${wheel_width}"/>
+        <sphere radius="${caster_radius}"/>
       </geometry>
       <material name="black">
-        <color rgba="0.1 0.1 0.1 1.0"/>
+        <color rgba="0 0 0 1"/>
       </material>
     </visual>
-    <inertial>
-      <origin xyz="0 0 0" rpy="${pi/2} 0 0"/>
-      <mass value="${wheel_mass}"/>
-      <inertia
-        ixx="${wheel_mass/12.0 * (3*wheel_radius*wheel_radius + wheel_width*wheel_width)}"
-        ixy="0.0"
-        ixz="0.0"
-        iyy="${wheel_mass/12.0 * (3*wheel_radius*wheel_radius + wheel_width*wheel_width)}"
-        iyz="0.0"
-        izz="${wheel_mass/2.0 * wheel_radius*wheel_radius}"/>
-    </inertial>
-  </link>
-  <!-- Right Wheel Joint -->
-  <joint name="$(arg robot_namespace)/right_wheel_joint" type="continuous">
-    <parent link="$(arg robot_namespace)/base_link"/>
-    <child link="$(arg robot_namespace)/right_wheel"/>
-    <origin xyz="${wheel_offset_x} -${wheel_offset_y} ${wheel_offset_z}" rpy="0 0 0"/>
-    <axis xyz="0 1 0"/>
-  </joint>
-  <!-- Caster Wheel Link -->
-  <link name="$(arg robot_namespace)/caster_wheel">
     <collision>
-      <origin xyz="0 0 0" rpy="0 0 0"/>
       <geometry>
         <sphere radius="${caster_radius}"/>
       </geometry>
     </collision>
+    <inertial>
+      <mass value="0.1"/>
+      <inertia ixx="0.001" ixy="0" ixz="0" iyy="0.001" iyz="0" izz="0.001"/>
+    </inertial>
+  </link>
+  <!-- Joints -->
+  <joint name="left_wheel_joint" type="continuous">
+    <parent link="base_link"/>
+    <child link="left_wheel"/>
+    <origin xyz="0 ${wheel_separation/2} ${wheel_offset_z}" rpy="-1.5708 0 0"/>
+    <axis xyz="0 0 1"/>
+  </joint>
+  <joint name="right_wheel_joint" type="continuous">
+    <parent link="base_link"/>
+    <child link="right_wheel"/>
+    <origin xyz="0 ${-wheel_separation/2} ${wheel_offset_z}" rpy="-1.5708 0 0"/>
+    <axis xyz="0 0 1"/>
+  </joint>
+  <joint name="front_caster_joint" type="fixed">
+    <parent link="base_link"/>
+    <child link="front_caster"/>
+    <origin xyz="${base_length/3} 0 ${-base_height/2}" rpy="0 0 0"/>
+  </joint>
+  <!-- Sensors -->
+  <link name="laser_link">
     <visual>
-      <origin xyz="0 0 0" rpy="0 0 0"/>
       <geometry>
-        <sphere radius="${caster_radius}"/>
+        <cylinder radius="0.025" length="0.05"/>
       </geometry>
       <material name="black">
-        <color rgba="0.1 0.1 0.1 1.0"/>
+        <color rgba="0 0 0 1"/>
       </material>
     </visual>
+    <collision>
+      <geometry>
+        <cylinder radius="0.025" length="0.05"/>
+      </geometry>
+    </collision>
     <inertial>
-      <origin xyz="0 0 0" rpy="0 0 0"/>
-      <mass value="${caster_mass}"/>
-      <inertia
-        ixx="${2.0*caster_mass*caster_radius*caster_radius/5.0}"
-        ixy="0.0"
-        ixz="0.0"
-        iyy="${2.0*caster_mass*caster_radius*caster_radius/5.0}"
-        iyz="0.0"
-        izz="${2.0*caster_mass*caster_radius*caster_radius/5.0}"/>
+      <mass value="0.1"/>
+      <inertia ixx="0.001" ixy="0" ixz="0" iyy="0.001" iyz="0" izz="0.001"/>
     </inertial>
   </link>
-  <!-- Caster Wheel Joint -->
-  <joint name="$(arg robot_namespace)/caster_wheel_joint" type="fixed">
-    <parent link="$(arg robot_namespace)/base_link"/>
-    <child link="$(arg robot_namespace)/caster_wheel"/>
-    <origin xyz="-${chassis_length/4} 0 -${caster_radius/2}" rpy="0 0 0"/>
+  <joint name="laser_joint" type="fixed">
+    <parent link="base_link"/>
+    <child link="laser_link"/>
+    <origin xyz="${base_length/2} 0 ${base_height/2}" rpy="0 0 0"/>
   </joint>
-  <!-- LiDAR Sensor Link -->
-  <link name="$(arg robot_namespace)/lidar_link">
+  <!-- Camera -->
+  <link name="camera_link">
+    <visual>
+      <geometry>
+        <box size="0.05 0.05 0.05"/>
+      </geometry>
+      <material name="black">
+        <color rgba="0 0 0 1"/>
+      </material>
+    </visual>
     <collision>
-      <origin xyz="0 0 0" rpy="0 0 0"/>
       <geometry>
-        <cylinder radius="0.05" length="0.04"/>
+        <box size="0.05 0.05 0.05"/>
       </geometry>
     </collision>
-    <visual>
-      <origin xyz="0 0 0" rpy="0 0 0"/>
-      <geometry>
-        <cylinder radius="0.05" length="0.04"/>
-      </geometry>
-      <material name="blue">
-        <color rgba="0.0 0.0 0.8 1.0"/>
-      </material>
-    </visual>
     <inertial>
       <mass value="0.1"/>
-      <origin xyz="0 0 0" rpy="0 0 0"/>
-      <inertia
-        ixx="0.001"
-        ixy="0.0"
-        ixz="0.0"
-        iyy="0.001"
-        iyz="0.0"
-        izz="0.001"/>
+      <inertia ixx="0.001" ixy="0" ixz="0" iyy="0.001" iyz="0" izz="0.001"/>
     </inertial>
   </link>
-  <!-- LiDAR Sensor Joint -->
-  <joint name="$(arg robot_namespace)/lidar_joint" type="fixed">
-    <parent link="$(arg robot_namespace)/base_link"/>
-    <child link="$(arg robot_namespace)/lidar_link"/>
-    <origin xyz="0 0 ${chassis_height + 0.02}" rpy="0 0 0"/>
+  <joint name="camera_joint" type="fixed">
+    <parent link="base_link"/>
+    <child link="camera_link"/>
+    <origin xyz="${base_length/2} 0 ${base_height}" rpy="0 0 0"/>
   </joint>
 </robot>
