Commit message: Add Gazebo-specific robot configurations

File: mars_robots/urdf/mars_robot.gazebo.xacro (robot description, xacro)
@@ -1,81 +1,44 @@
 <?xml version="1.0"?>
 <robot xmlns:xacro="http://www.ros.org/wiki/xacro">
-  <!-- Define properties needed for gazebo plugins -->
-  <xacro:property name="wheel_radius" value="0.1" />
-  <xacro:property name="wheel_offset_y" value="0.175" />
-  <!-- Gazebo-specific robot configuration -->
-  <gazebo reference="$(arg robot_namespace)/base_link">
-    <material>Gazebo/Red</material>
+  <!-- Gazebo plugin for ROS Control -->
+  <gazebo>
+    <plugin name="gazebo_ros_control" filename="libgazebo_ros_control.so">
+      <robotNamespace>/</robotNamespace>
+      <robotSimType>gazebo_ros_control/DefaultRobotHWSim</robotSimType>
+      <legacyModeNS>true</legacyModeNS>
+    </plugin>
   </gazebo>
-  <gazebo reference="$(arg robot_namespace)/left_wheel">
-    <material>Gazebo/Black</material>
-    <mu1>1.0</mu1>
-    <mu2>1.0</mu2>
-    <kp>1000000.0</kp>
-    <kd>100.0</kd>
-    <minDepth>0.001</minDepth>
-    <maxVel>1.0</maxVel>
-  </gazebo>
-  <gazebo reference="$(arg robot_namespace)/right_wheel">
-    <material>Gazebo/Black</material>
-    <mu1>1.0</mu1>
-    <mu2>1.0</mu2>
-    <kp>1000000.0</kp>
-    <kd>100.0</kd>
-    <minDepth>0.001</minDepth>
-    <maxVel>1.0</maxVel>
-  </gazebo>
-  <gazebo reference="$(arg robot_namespace)/caster_wheel">
-    <material>Gazebo/Black</material>
-    <mu1>0.1</mu1>
-    <mu2>0.1</mu2>
-    <kp>1000000.0</kp>
-    <kd>100.0</kd>
-    <minDepth>0.001</minDepth>
-    <maxVel>1.0</maxVel>
-  </gazebo>
-  <gazebo reference="$(arg robot_namespace)/lidar_link">
-    <material>Gazebo/Blue</material>
-  </gazebo>
-  <!-- Differential Drive Controller Plugin -->
+  <!-- Differential drive controller -->
   <gazebo>
     <plugin name="differential_drive_controller" filename="libgazebo_ros_diff_drive.so">
-      <!-- Plugin update rate -->
-      <update_rate>30</update_rate>
-      <!-- Left/Right wheel joints -->
-      <left_joint>$(arg robot_namespace)/left_wheel_joint</left_joint>
-      <right_joint>$(arg robot_namespace)/right_wheel_joint</right_joint>
-      <!-- Robot characteristics -->
-      <wheel_separation>${wheel_offset_y * 2}</wheel_separation>
-      <wheel_diameter>${wheel_radius * 2}</wheel_diameter>
-      <!-- Limits -->
-      <max_wheel_acceleration>1.0</max_wheel_acceleration>
-      <max_wheel_torque>20</max_wheel_torque>
-      <!-- Command topic -->
-      <command_topic>cmd_vel</command_topic>
-      <!-- Odometry output -->
-      <publish_odom>true</publish_odom>
-      <publish_odom_tf>true</publish_odom_tf>
-      <publish_wheel_tf>true</publish_wheel_tf>
-      <odometry_topic>odom</odometry_topic>
-      <odometry_frame>$(arg robot_namespace)/odom</odometry_frame>
-      <robot_base_frame>$(arg robot_namespace)/base_footprint</robot_base_frame>
-      <!-- Publishers -->
-      <ros>
-        <remapping>odom:=odom</remapping>
-        <remapping>cmd_vel:=cmd_vel</remapping>
-      </ros>
+      <updateRate>50</updateRate>
+      <leftJoint>left_wheel_joint</leftJoint>
+      <rightJoint>right_wheel_joint</rightJoint>
+      <wheelSeparation>${wheel_separation}</wheelSeparation>
+      <wheelDiameter>${2*wheel_radius}</wheelDiameter>
+      <wheelAcceleration>1.0</wheelAcceleration>
+      <wheelTorque>20</wheelTorque>
+      <commandTopic>cmd_vel</commandTopic>
+      <odometryTopic>odom</odometryTopic>
+      <odometryFrame>odom</odometryFrame>
+      <robotBaseFrame>base_link</robotBaseFrame>
+      <publishWheelTF>true</publishWheelTF>
+      <publishOdomTF>true</publishOdomTF>
+      <publishWheelJointState>true</publishWheelJointState>
+      <legacyMode>false</legacyMode>
+      <odometrySource>world</odometrySource>
+      <publishTf>true</publishTf>
     </plugin>
   </gazebo>
-  <!-- LiDAR Sensor -->
-  <gazebo reference="$(arg robot_namespace)/lidar_link">
-    <sensor type="ray" name="lidar">
+  <!-- Laser Scanner -->
+  <gazebo reference="laser_link">
+    <sensor type="ray" name="laser">
       <pose>0 0 0 0 0 0</pose>
-      <update_rate>5</update_rate>
       <visualize>true</visualize>
+      <update_rate>10</update_rate>
       <ray>
         <scan>
           <horizontal>
-            <samples>120</samples>
+            <samples>360</samples>
             <resolution>1</resolution>
             <min_angle>-3.14159</min_angle>
@@ -85,5 +48,5 @@
         <range>
           <min>0.10</min>
-          <max>2.0</max>
+          <max>10.0</max>
           <resolution>0.01</resolution>
         </range>
@@ -94,23 +57,69 @@
         </noise>
       </ray>
-      <plugin name="lidar_controller" filename="libgazebo_ros_ray_sensor.so">
+      <plugin name="laser_controller" filename="libgazebo_ros_ray_sensor.so">
         <ros>
+          <namespace>/</namespace>
           <remapping>~/out:=scan</remapping>
         </ros>
         <output_type>sensor_msgs/LaserScan</output_type>
-        <frame_name>$(arg robot_namespace)/lidar_link</frame_name>
+        <frame_name>laser_link</frame_name>
       </plugin>
     </sensor>
   </gazebo>
-  <!-- Joint State Publisher -->
-  <gazebo>
-    <plugin name="joint_state_publisher" filename="libgazebo_ros_joint_state_publisher.so">
-      <ros>
-        <remapping>~/out:=joint_states</remapping>
-      </ros>
-      <update_rate>30</update_rate>
-      <joint_name>$(arg robot_namespace)/left_wheel_joint</joint_name>
-      <joint_name>$(arg robot_namespace)/right_wheel_joint</joint_name>
-    </plugin>
+  <!-- Camera -->
+  <gazebo reference="camera_link">
+    <sensor type="camera" name="camera">
+      <update_rate>30.0</update_rate>
+      <camera name="head">
+        <horizontal_fov>1.3962634</horizontal_fov>
+        <image>
+          <width>800</width>
+          <height>600</height>
+          <format>R8G8B8</format>
+        </image>
+        <clip>
+          <near>0.02</near>
+          <far>300</far>
+        </clip>
+        <noise>
+          <type>gaussian</type>
+          <mean>0.0</mean>
+          <stddev>0.007</stddev>
+        </noise>
+      </camera>
+      <plugin name="camera_controller" filename="libgazebo_ros_camera.so">
+        <alwaysOn>true</alwaysOn>
+        <updateRate>0.0</updateRate>
+        <cameraName>camera</cameraName>
+        <imageTopicName>image_raw</imageTopicName>
+        <cameraInfoTopicName>camera_info</cameraInfoTopicName>
+        <frameName>camera_link</frameName>
+        <hackBaseline>0.07</hackBaseline>
+        <distortionK1>0.0</distortionK1>
+        <distortionK2>0.0</distortionK2>
+        <distortionK3>0.0</distortionK3>
+        <distortionT1>0.0</distortionT1>
+        <distortionT2>0.0</distortionT2>
+      </plugin>
+    </sensor>
+  </gazebo>
+  <!-- Material colors -->
+  <gazebo reference="base_link">
+    <material>Gazebo/Red</material>
+  </gazebo>
+  <gazebo reference="left_wheel">
+    <material>Gazebo/Black</material>
+    <mu1>0.8</mu1>
+    <mu2>0.8</mu2>
+  </gazebo>
+  <gazebo reference="right_wheel">
+    <material>Gazebo/Black</material>
+    <mu1>0.8</mu1>
+    <mu2>0.8</mu2>
+  </gazebo>
+  <gazebo reference="front_caster">
+    <material>Gazebo/Black</material>
+    <mu1>0.0</mu1>
+    <mu2>0.0</mu2>
   </gazebo>
 </robot>
